File: flexglove.sch (EAGLE design)
At the start: 11 parts, among them J1 USB_A_SMT_FEMALE, U2 FT232RL

Commit message: parts
Parts:
- added C2: 0.1uF, SparkFun-Capacitors:0.1UF-0603-25V-5%
- added C5: 22UF-1210-16V-20%, SparkFun-Capacitors:22UF-1210-16V-20%
- added C6: 470pF, SparkFun-Capacitors:470PF-0603-50V-5%
- added D3: 1A/40V/500mV, SparkFun-DiscreteSemi:DIODE-SCHOTTKY-SS14
- added J3, J4, J5, J6, J7, J8, J9: (no value), SparkFun-Connectors:CONN_02
- added M1: MOTOR10MM, SparkFun-Electromechanical:MOTOR10MM
- added Q1: 600mA/40V, SparkFun-DiscreteSemi:TRANS_NPN-MMBT2222AL
- added R10, R11, R12, R3, R4, R5, R6, R7, R8, R9: 1k, SparkFun-Resistors:1KOHM-0603-1/10W-1%
- added U1: MIC5219 3.3V, SparkFun-IC-Power:V_REG_MIC52193.3V
- J2: device SparkFun-Connectors:CONN_05JST -> SparkFun-Connectors:CONN_02
Connections:
- new net 3V3_EN: U$1.PT7, U1.EN
- new net BUZ_PWM: R3.1, U$1.PT3
- new net N$10: J9.2, R12.1, U$1.AN7
- new net N$11: Q1.B, R3.2, R4.2
- new net N$12: C4.1, U2.3V3OUT
- new net N$13: C2.2, D3.A, M1.-, Q1.C
- new net N$14: C6.1, U1.BP
- new net N$8: J4.2, R7.1, U$1.AN2
- new net N$9: J8.2, R11.1, U$1.AN6
- net 3.3V: now also C2.1, C5.1, D3.C, M1.+, U1.OUT; no longer C4.1, U2.3V3OUT
- net 5V: now also R10.2, R11.2, R12.2, R5.2, R6.2, R7.2, R8.2, R9.2, U1.IN
- net GND: now also C5.2, C6.2, J2.1, J3.1, J4.1, J5.1, J6.1, J7.1, J8.1, J9.1, Q1.E, R4.1, U1.GND
- net N$3: now also J2.2, R5.1, U$1.AN0; no longer J2.5, U$1.AN1
- net N$4: now also J3.2, R6.1, U$1.AN1; no longer J2.4, U$1.AN2
- net N$5: now also J5.2, R8.1; no longer J2.3
- net N$6: now also J6.2, R9.1; no longer J2.2
- net N$7: now also J7.2, R10.1; no longer J2.1
